Commit message: Moving robot

File: lab2/urdf/moving_robot.xacro (robot description, xacro)
@@ -14,10 +14,11 @@
     <xacro:property name="base_radius" value="0.1"/>
     <!-- macros -->
-    <xacro:macro name="default_joint" params="joint_params number">
-        <joint name="link${number-1}_to_link_${number}" type="fixed">
+    <xacro:macro name="default_joint" params="joint_params number min max">
+        <joint name="link${number-1}_to_link_${number}" type="revolute">
             <parent link="link_${number-1}"/>
             <child link="link_${number}"/>
             <origin xyz="${joint_params['xyz']}" rpy="${joint_params['rpy']}"/>
             <axis xyz="0.0 0.0 1.0"/>
+            <limit effort="1000.0" lower="${min}" upper="${max}" velocity="0.5"/>
         </joint>
     </xacro:macro>
@@ -47,7 +48,7 @@
         <visual>
             <geometry>
-                <cylinder length="${base_length}" radius="${base_radius}"/>
+                <box size="${link_width} ${link_width} ${link_width}"/>
             </geometry>
-            <origin xyz="0 0 ${base_length/-2}"/>
+            <origin xyz="0 0 0"/>
             <material name="green"/>
         </visual>
@@ -64,11 +65,12 @@
         </visual>
     </link>
-    <joint name="base_to_link_1" type="fixed">
+    <joint name="base_to_link_1" type="revolute">
         <parent link="base_link"/>
         <child link="link_1"/>
         <origin xyz="${joint1_params['xyz']}" rpy="${joint1_params['rpy']}"/>
         <axis xyz="0 0 1"/>
+        <limit effort="1000.0" lower="-3.1415" upper="3.1415" velocity="0.5"/>
     </joint>
-    <xacro:default_joint joint_params="${joint2_params}" number="2"/>
-    <xacro:default_joint joint_params="${joint3_params}" number="3"/>
+    <xacro:default_joint joint_params="${joint2_params}" number="2" min="-3.14" max="0"/>
+    <xacro:default_joint joint_params="${joint3_params}" number="3" min="-1.57" max="1.57"/>
 </robot>

File: lab2/urdf/static_robot_generated.urdf (robot description, URDF)
Before this commit: robot lab2_robot, 4 links, 3 joints
Links:
- removed link link1
- removed link link2
- removed link link3
- added link link_1; visual box size=0 0.1 0.1
- added link link_2; visual box size=1 0.1 0.1
- added link link_3; visual cylinder length=0.2 radius=0.05
- link base_link: geometry visual cylinder length=0.1 radius=0.1
Joints:
- removed joint joint1
- removed joint joint2
- removed joint joint3
- added joint base_to_link_1: type fixed, parent base_link, child link_1, origin xyz=0.0 0.0 0.0 rpy=0.0 -0.0 0.0, axis 0 0 1
- added joint link1_to_link_2: type fixed, parent link_1, child link_2, origin xyz=0.0 0.0 0.0 rpy=-1.57 -0.0 0.0, axis 0.0 0.0 1.0
- added joint link2_to_link_3: type fixed, parent link_2, child link_3, origin xyz=1.0 0.0 0.0 rpy=0.0 -0.0 0.0, axis 0.0 0.0 1.0
